File: _autosave-Силовая плата.kicad_pcb (KiCad board)
At the start: 2 copper layers, 75 x 75 mm, 9 parts, among them Q1 BSP89, Q2 BSP89, Q3 BSP89, Q4 BSP89, Q5 BSP89, Q6 BSP89, U1 HIP2100_SOIC, U2 HIP2100_SOIC, U3 HIP2100_SOIC

Commit message: Базовый вариант
Parts:
- U1, U2, U3: moved to B.Cu
- moved U3 113.4 mm to (170.1, 73.5)
- moved U2 85.4 mm to (145.3, 73.5)
- moved U1 59.2 mm to (118.6, 73.2), turned to 90 degrees
- moved Q2 0.47 mm to (127.0, 81.3)
Routing:
- net G4: track 0.00 -> 3.30 mm, vias 0 -> 1
- net G6: track 0.00 -> 3.30 mm, vias 0 -> 1
- net G2: track 0.00 -> 3.04 mm, vias 0 -> 1
- added copper zone on F.Cu, net B
- added copper zone on F.Cu, net C

Commit message: Базовый вариант
Parts:
- U1, U2, U3: footprint Package_DFN_QFN:DFN-8-1EP_3x3mm_P0.5mm_EP1.65x2.38mm -> Package_SO:SOIC-8_3.9x4.9mm_P1.27mm; moved to F.Cu
- moved U1 69.9 mm to (180.3, 106.1)
- moved U3 53.5 mm to (127.6, 106.1)
- moved U2 33.8 mm to (154.3, 106.1)
Routing:
- net G6: track 3.30 -> 40.7 mm
- net G4: track 3.30 -> 40.2 mm
- net G2: track 3.04 -> 39.6 mm
- net G3: track 0.00 -> 20.4 mm, vias 0 -> 1
- net G5: track 0.00 -> 19.4 mm, vias 0 -> 1
- net G1: track 0.00 -> 18.9 mm, vias 0 -> 1
- net C: vias 0 -> 12
- net B: vias 0 -> 12
- net A: vias 0 -> 12
- net +12V: vias 0 -> 11
- added copper zone on B.Cu, net +12V
- added copper zone on B.Cu, net A
- added copper zone on In1.Cu, net A
- added copper zone on In2.Cu, net A
- added copper zone on In3.Cu, net A
- added copper zone on In4.Cu, net A
- added copper zone on B.Cu, net B
- added copper zone on In1.Cu, net B
- added copper zone on In2.Cu, net B
- added copper zone on In3.Cu, net B
- added copper zone on In4.Cu, net B
- added copper zone on B.Cu, net C
- added copper zone on In1.Cu, net C
- added copper zone on In2.Cu, net C
- added copper zone on In3.Cu, net C
- added copper zone on In4.Cu, net C
- added copper zone on In1.Cu, net GND
- added copper zone on In2.Cu, net GND
- added copper zone on In3.Cu, net GND
- added copper zone on In4.Cu, net GND
Other:
- copper layers 2 -> 6
