File: Силовая плата.kicad_pcb (KiCad board)
At the start: 6 copper layers, 68 x 66.7 mm, 66 parts, among them J1 Conn_01x01, J2 Conn_01x01, J3 Conn_01x01, J4 Conn_01x01, J5 Conn_01x01, J6 2-338069-0, Q1 BSP89, Q2 BSP89, Q3 BSP89, Q4 BSP89, Q5 BSP89, Q6 BSP89, U1 IRS21867S, U2 IRS21867S, U3 IRS21867S

Commit message: Добавил шунты
Parts:
- removed C43, C44, C45, C46, C47, C48: 4.7u, Capacitor_SMD:C_1206_3216Metric_Pad1.33x1.80mm_HandSolder
- removed U1, U2, U3: IRS21867S, Package_SO:SOIC-8_3.9x4.9mm_P1.27mm
- added C10: 0.1u, Capacitor_SMD:C_0805_2012Metric_Pad1.18x1.45mm_HandSolder, F.Cu at (170.2, 121.5)
- added C2: 1400m, Capacitor_THT:CP_Axial_L30.0mm_D18.0mm_P35.00mm_Horizontal, F.Cu at (1.48, 31.5)
- added C3: 1400m, Capacitor_THT:CP_Axial_L30.0mm_D18.0mm_P35.00mm_Horizontal, F.Cu at (54.3, 124.5)
- added D4: ADP3110A, Package_DFN_QFN:DFN-8-1EP_3x3mm_P0.65mm_EP1.7x2.05mm, F.Cu at (133.6, 108.0)
- added D5: D_Small, Diode_SMD:D_SOD-323, F.Cu at (161.3, 104.8)
- added D6: ADP3110A, Package_DFN_QFN:DFN-8-1EP_3x3mm_P0.65mm_EP1.7x2.05mm, F.Cu at (165.5, 108.0)
- added R21: 10k, Resistor_SMD:R_0805_2012Metric_Pad1.20x1.40mm_HandSolder, F.Cu at (189.0, 93.3)
- added R22: 10k, Resistor_SMD:R_0805_2012Metric_Pad1.20x1.40mm_HandSolder, F.Cu at (189.0, 96.3)
- added R23: 10k, Resistor_SMD:R_0805_2012Metric_Pad1.20x1.40mm_HandSolder, F.Cu at (189.0, 99.2)
- added R24: R, Resistor_SMD:R_2512_6332Metric_Pad1.40x3.35mm_HandSolder, B.Cu at (174.0, 128.1)
- added R25: R, Resistor_SMD:R_2512_6332Metric_Pad1.40x3.35mm_HandSolder, B.Cu at (174.0, 132.6)
- added R26: R, Resistor_SMD:R_2512_6332Metric_Pad1.40x3.35mm_HandSolder, B.Cu at (174.0, 123.7)
- added R27: R, Resistor_SMD:R_2512_6332Metric_Pad1.40x3.35mm_HandSolder, B.Cu at (173.9, 119.2)
- added R28: R, Resistor_SMD:R_2512_6332Metric_Pad1.40x3.35mm_HandSolder, B.Cu at (165.7, 117.5)
- added R29: R, Resistor_SMD:R_2512_6332Metric_Pad1.40x3.35mm_HandSolder, B.Cu at (129.5, 132.6)
- added R30: R, Resistor_SMD:R_2512_6332Metric_Pad1.40x3.35mm_HandSolder, B.Cu at (129.5, 119.2)
- added R31: R, Resistor_SMD:R_2512_6332Metric_Pad1.40x3.35mm_HandSolder, B.Cu at (137.8, 117.5)
- added R32: R, Resistor_SMD:R_2512_6332Metric_Pad1.40x3.35mm_HandSolder, B.Cu at (142.2, 117.5)
- added R34: R, Resistor_SMD:R_2512_6332Metric_Pad1.40x3.35mm_HandSolder, B.Cu at (146.7, 117.5)
- added R35: R, Resistor_SMD:R_2512_6332Metric_Pad1.40x3.35mm_HandSolder, B.Cu at (161.3, 117.5)
- added R36: R, Resistor_SMD:R_2512_6332Metric_Pad1.40x3.35mm_HandSolder, B.Cu at (156.8, 117.5)
- added R37: R, Resistor_SMD:R_2512_6332Metric_Pad1.40x3.35mm_HandSolder, B.Cu at (129.5, 123.7)
- added R38: R, Resistor_SMD:R_2512_6332Metric_Pad1.40x3.35mm_HandSolder, B.Cu at (129.5, 128.1)
- added U6: AD8210, Package_SO:SOIC-8_3.9x4.9mm_P1.27mm, F.Cu at (175.3, 121.3)
- C4, C6, C8: value C_Small -> 10u
- D3: value D_Small -> ADP3110A; footprint Diode_SMD:D_SOD-323 -> Package_DFN_QFN:DFN-8-1EP_3x3mm_P0.65mm_EP1.7x2.05mm
- moved C1 100.6 mm to (229.8, 162.6)
- moved C33 62.1 mm to (125.1, 125.7), turned to -90 degrees
- moved C25 61.7 mm to (125.1, 130.8), turned to 90 degrees
- moved C26 60.0 mm to (125.1, 105.4), turned to -90 degrees
- moved C36 59.9 mm to (179.7, 95.2), turned to -90 degrees
- moved C27 59.7 mm to (125.1, 110.5), turned to 90 degrees
- moved C24 58.7 mm to (127.6, 125.7), turned to -90 degrees
- moved C37 56.7 mm to (177.2, 95.2), turned to -90 degrees
- moved C35 54.5 mm to (174.6, 100.3), turned to 90 degrees
- moved C15 53.8 mm to (125.1, 120.7), turned to 90 degrees
- moved C38 53.6 mm to (174.6, 95.2), turned to -90 degrees
- moved C14 50.7 mm to (127.6, 120.7), turned to 90 degrees
- moved C28 50.2 mm to (130.2, 100.3), turned to 90 degrees
- moved C16 22.9 mm to (127.6, 130.8), turned to 90 degrees
- moved D3 21.8 mm to (149.7, 108.0), turned to 0 degrees
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Connections:
- C4 pad 1: Net-(U1-COM) -> GND
- C4 pad 2: Net-(D1-A) -> +12V
- C5 pad 1: Net-(D1-K) -> A
- C5 pad 2: Net-(U1-VS) -> Net-(D1-K)
- C6 pad 1: Net-(U2-COM) -> GND
- C6 pad 2: Net-(D2-A) -> +12V
- C7 pad 1: Net-(D2-K) -> B
- C7 pad 2: Net-(U2-VS) -> Net-(D2-K)
- C8 pad 1: Net-(U3-COM) -> GND
- C8 pad 2: Net-(D3-A) -> +12V
- C9 pad 1: Net-(D3-K) -> C
- D1 pad 2: Net-(D1-A) -> +12V
- D2 pad 2: Net-(D2-A) -> +12V
- D3 pad 1: Net-(D3-K) -> Net-(D2-K)
- D3 pad 2: Net-(D3-A) -> IN_B
- J2 pad 1: GND -> -BATT
- J6 pad 1: HIN_A -> IN_A
- J6 pad 10: LIN_B -> IN_B
- J6 pad 11: HIN_B -> unconnected-(J6-Pad11)
- J6 pad 17: unconnected-(J6-Pad17) -> IN_C
- J6 pad 19: LIN_C -> DC_Measure
- J6 pad 2: LIN_A -> Enable
- J6 pad 20: HIN_C -> +5V
- R15 pad 1: Net-(U2-HO) -> Net-(D3-DRVH)
- R16 pad 1: Net-(U2-LO) -> Net-(D3-DRVL)
Routing:
- net GND: track 118.5 -> 21.1 mm, vias 50 -> 25
- net HIN_A: track 25.0 -> 0.00 mm, vias 2 -> 0
- net LIN_A: track 24.3 -> 0.00 mm, vias 2 -> 0
- net C: track 0.00 -> 22.6 mm, vias 0 -> 3
- net A: track 0.00 -> 22.6 mm, vias 0 -> 3
- net B: track 0.00 -> 21.7 mm, vias 0 -> 3
- net G5: track 4.43 -> 22.8 mm, vias 0 -> 2
- net G6: track 17.7 -> 35.3 mm
- net G3: track 4.49 -> 22.0 mm, vias 0 -> 2
- net G1: track 4.44 -> 21.4 mm, vias 0 -> 2
- net G4: track 17.6 -> 34.5 mm
- net +12V: track 0.00 -> 16.5 mm, vias 0 -> 6
- net HIN_C: track 16.5 -> 0.00 mm, vias 2 -> 0
- net G2: track 17.7 -> 33.9 mm
- net LIN_B: track 16.2 -> 0.00 mm, vias 2 -> 0
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- added copper zone on B.Cu, net -BATT
- removed copper zone on B.Cu, net +24V
- removed copper zone on In1.Cu, net +24V
- removed copper zone on In2.Cu, net GND
Other:
- board size 68 x 66.7 mm -> 60.4 x 76.3 mm

Commit message: Для презентации
Parts:
- removed C20, C26, C28, C39, C40, C41, C42: 4.7u, Capacitor_SMD:C_1206_3216Metric_Pad1.33x1.80mm_HandSolder
- removed C3: 1400m, Capacitor_THT:CP_Axial_L30.0mm_D18.0mm_P35.00mm_Horizontal
- removed R21, R22, R23: 10k, Resistor_SMD:R_0805_2012Metric_Pad1.20x1.40mm_HandSolder
- removed R24, R25, R26, R27, R28, R29, R30, R31, R32, R35, R36, R37, R38: R, Resistor_SMD:R_2512_6332Metric_Pad1.40x3.35mm_HandSolder
- C1: footprint Capacitor_THT:CP_Axial_L18.0mm_D8.0mm_P25.00mm_Horizontal -> Capacitor_THT:CP_Axial_L30.0mm_D18.0mm_P35.00mm_Horizontal
- R34: footprint Resistor_SMD:R_2512_6332Metric_Pad1.40x3.35mm_HandSolder -> Resistor_SMD:R_Shunt_Vishay_WSR2_WSR3; moved to F.Cu
- moved C2 187.5 mm to (134.3, 163.8)
- moved C1 97.2 mm to (134.3, 144.8)
- moved R34 26.1 mm to (127.0, 100.3)
- moved C5 4.08 mm to (137.8, 104.1)
- moved D1 4.08 mm to (133.3, 104.1)
Connections:
- J2 pad 1: -BATT -> GND
- Q1 pad 2: +24V -> Net-(Q1-D)
- Q3 pad 2: +24V -> Net-(Q1-D)
- Q5 pad 2: +24V -> Net-(Q1-D)
- R34 pad 1: -BATT -> +24V
- R34 pad 2: GND -> Net-(Q1-D)
Routing:
- net A: track 22.6 -> 27.3 mm
- net Net-(D1-K): track 4.80 -> 6.13 mm
- removed copper zone on B.Cu, net -BATT

Commit message: Стартовый вариант
Parts:
- removed C34, C35, C36, C37, C38: 4.7u, Capacitor_SMD:C_1206_3216Metric_Pad1.33x1.80mm_HandSolder
- removed J1, J2: Conn_01x01, Connector_My:Power_Wire
- removed J6: 2-338069-0, Connector_My:2-338069-0
- added C11: 56p, Capacitor_SMD:C_0805_2012Metric_Pad1.18x1.45mm_HandSolder, F.Cu at (84.5, 92.1)
- added C12: 56p, Capacitor_SMD:C_0805_2012Metric_Pad1.18x1.45mm_HandSolder, F.Cu at (82.5, 98.4)
- added C20: 4.7u, Capacitor_SMD:C_1206_3216Metric_Pad1.33x1.80mm_HandSolder, F.Cu at (89.5, 122.6)
- added C26: 4.7u, Capacitor_SMD:C_1206_3216Metric_Pad1.33x1.80mm_HandSolder, F.Cu at (87.0, 122.6)
- added C28: 4.7u, Capacitor_SMD:C_1206_3216Metric_Pad1.33x1.80mm_HandSolder, F.Cu at (92.1, 117.5)
- added C3: 0.1u, Capacitor_SMD:C_0805_2012Metric_Pad1.18x1.45mm_HandSolder, F.Cu at (86.4, 96.5)
- added R1: R, Shunt_My:TLRS1050, F.Cu at (78.1, 103.1)
- added R2: 120, Resistor_SMD:R_0805_2012Metric_Pad1.20x1.40mm_HandSolder, F.Cu at (81.9, 92.1)
- added R21: 10k, Resistor_SMD:R_0805_2012Metric_Pad1.20x1.40mm_HandSolder, F.Cu at (78.1, 94.9)
- added R22: 10k, Resistor_SMD:R_0805_2012Metric_Pad1.20x1.40mm_HandSolder, F.Cu at (88.9, 94.6)
- added R23: 10k, Resistor_SMD:R_0805_2012Metric_Pad1.20x1.40mm_HandSolder, F.Cu at (82.9, 88.3)
- added R3: 120, Resistor_SMD:R_0805_2012Metric_Pad1.20x1.40mm_HandSolder, F.Cu at (92.1, 102.9)
- added R4: 120, Resistor_SMD:R_0805_2012Metric_Pad1.20x1.40mm_HandSolder, F.Cu at (92.1, 107.3)
- added R5: 120, Resistor_SMD:R_0805_2012Metric_Pad1.20x1.40mm_HandSolder, F.Cu at (87.0, 99.7)
- added U1: LMV7239M5, Package_TO_SOT_SMD:SOT-353_SC-70-5, F.Cu at (82.5, 95.9)
- R13, R14, R15, R16, R17, R18: footprint Resistor_SMD:R_1206_3216Metric_Pad1.30x1.75mm_HandSolder -> Resistor_SMD:R_0805_2012Metric_Pad1.20x1.40mm_HandSolder
- R34: footprint Resistor_SMD:R_Shunt_Vishay_WSR2_WSR3 -> Shunt_My:TLRS1050
- moved J5 121.9 mm to (53.3, 82.4)
- moved Q5 106.1 mm to (60.7, 102.3)
- moved Q6 105.8 mm to (61.6, 85.7), turned to 180 degrees
- moved R18 104.3 mm to (68.6, 92.7), turned to 180 degrees
- moved R17 103.5 mm to (68.6, 95.2), turned to 180 degrees
- moved C31 101.1 mm to (79.4, 117.5)
- moved C32 101.1 mm to (76.8, 117.5)
- moved C9 97.4 mm to (68.6, 97.8), turned to 0 degrees
- moved C30 94.3 mm to (87.0, 117.5), turned to -90 degrees
- moved C29 94.3 mm to (84.5, 117.5), turned to -90 degrees
- moved C8 93.7 mm to (74.3, 90.8), turned to 0 degrees
- moved D6 92.7 mm to (73.9, 94.0), turned to 180 degrees
- moved U6 91.2 mm to (85.1, 107.3), turned to -90 degrees
- moved D5 87.9 mm to (73.7, 97.8), turned to 0 degrees
- moved C10 81.9 mm to (89.5, 107.3), turned to 90 degrees
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Connections:
- C1 pad 1: +24V -> Shunt_1
- C14 pad 1: +24V -> Shunt_1
- C15 pad 1: +24V -> Shunt_1
- C16 pad 1: +24V -> Shunt_1
- C17 pad 1: +24V -> Shunt_1
- C18 pad 1: +24V -> Shunt_1
- C19 pad 1: +24V -> Shunt_1
- C2 pad 1: +24V -> Shunt_1
- C21 pad 1: +24V -> Shunt_1
- C22 pad 1: +24V -> Shunt_1
- C23 pad 1: +24V -> Shunt_1
- C24 pad 1: +24V -> Shunt_1
- C25 pad 1: +24V -> Shunt_1
- C27 pad 1: +24V -> Shunt_1
- C29 pad 1: +24V -> Shunt_1
- C30 pad 1: +24V -> Shunt_1
- C31 pad 1: +24V -> Shunt_1
- C32 pad 1: +24V -> Shunt_1
- C33 pad 1: +24V -> Shunt_1
- Q1 pad 2: Net-(Q1-D) -> Shunt_2
- Q3 pad 2: Net-(Q1-D) -> Shunt_2
- Q5 pad 2: Net-(Q1-D) -> Shunt_2
- R34 pad 1: +24V -> Shunt_1
- R34 pad 2: Net-(Q1-D) -> Shunt_2
- U6 pad 1: -BATT -> Shunt_2
- U6 pad 8: GND -> Shunt_1
Routing:
- net GND: track 21.1 -> 79.9 mm, vias 25 -> 42
- net G6: track 35.3 -> 5.12 mm, vias 2 -> 0
- net G4: track 34.5 -> 5.02 mm, vias 2 -> 0
- net G2: track 33.9 -> 4.92 mm, vias 2 -> 0
- net A: track 27.3 -> 1.30 mm, vias 3 -> 11
- net Enable: track 5.30 -> 27.7 mm, vias 3 -> 0
- net C: track 22.6 -> 1.32 mm, vias 3 -> 11
- net Net-(U1-+): track 0.00 -> 20.6 mm, vias 0 -> 2
- net B: track 21.7 -> 1.24 mm, vias 3 -> 11
- net G5: track 22.8 -> 4.58 mm, vias 2 -> 0
- net G3: track 22.0 -> 4.58 mm, vias 2 -> 0
- net G1: track 21.4 -> 4.66 mm, vias 2 -> 0
- net DC_Measure: track 0.00 -> 12.1 mm, vias 0 -> 2
- net Shunt_1: track 0.00 -> 12.0 mm
- net Shunt_2: track 0.00 -> 12.0 mm, vias 0 -> 99
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- added copper zone on In1.Cu, net GND
- added copper zone on In2.Cu, net GND
- added copper zone on In3.Cu, net GND
- added copper zone on In4.Cu, net GND
- added copper zone on B.Cu, net Shunt_1
- added copper zone on F.Cu, net Shunt_1
- added copper zone on In1.Cu, net Shunt_1
- added copper zone on In2.Cu, net Shunt_1
- added copper zone on In3.Cu, net Shunt_1
- added copper zone on In4.Cu, net Shunt_1
- added copper zone on B.Cu, net Shunt_2
- added copper zone on F.Cu, net Shunt_2
- added copper zone on In1.Cu, net Shunt_2
- added copper zone on In2.Cu, net Shunt_2
- added copper zone on In3.Cu, net Shunt_2
- added copper zone on In4.Cu, net Shunt_2
- removed copper zone on F.Cu, net +24V
Other:
- board size 60.4 x 76.3 mm -> 65.7 x 72.2 mm

Commit message: Стартовая версия
Parts:
- removed C22, C23, C24, C25, C26, C27, C28, C29, C30, C31, C32, C33: 4.7u, Capacitor_SMD:C_1206_3216Metric_Pad1.33x1.80mm_HandSolder
- removed R22, R23: 10k, Resistor_SMD:R_0805_2012Metric_Pad1.20x1.40mm_HandSolder
- added J6: Conn_02x04_Odd_Even, Connector_PinHeader_2.54mm:PinHeader_2x04_P2.54mm_Vertical, F.Cu at (90.8, 113.0)
- added R10: 10k, Resistor_SMD:R_0805_2012Metric_Pad1.20x1.40mm_HandSolder, B.Cu at (68.6, 97.2)
- added R11: 10k, Resistor_SMD:R_0805_2012Metric_Pad1.20x1.40mm_HandSolder, B.Cu at (70.5, 87.9)
- added R6: 10k, Resistor_SMD:R_0805_2012Metric_Pad1.20x1.40mm_HandSolder, B.Cu at (81.3, 77.8)
- added R7: 10k, Resistor_SMD:R_0805_2012Metric_Pad1.20x1.40mm_HandSolder, B.Cu at (90.8, 81.9)
- added R8: 10k, Resistor_SMD:R_0805_2012Metric_Pad1.20x1.40mm_HandSolder, B.Cu at (99.1, 92.7)
- added R9: 10k, Resistor_SMD:R_0805_2012Metric_Pad1.20x1.40mm_HandSolder, B.Cu at (94.0, 102.2)
- C10, C11, C12, C3, R2, R21, R3, R4, R5, U1, U6: moved to B.Cu
- moved R2 15.4 mm to (91.4, 104.1)
- moved C10 11.4 mm to (78.1, 106.7), turned to 180 degrees
- moved C16 10.4 mm to (85.1, 118.4), turned to -90 degrees
- moved R21 9.55 mm to (86.4, 99.7), turned to -90 degrees
- moved C15 9.24 mm to (82.5, 118.4), turned to -90 degrees
- moved U1 9.09 mm to (86.4, 104.1), turned to 90 degrees
- moved C11 8.82 mm to (88.9, 99.7), turned to 90 degrees
- moved R34 8.51 mm to (73.9, 111.1), turned to 90 degrees
- moved R5 8.28 mm to (82.5, 106.7), turned to 180 degrees
- moved C3 8.03 mm to (88.9, 104.1)
- moved U6 7.67 mm to (78.1, 110.5), turned to 0 degrees
- moved R3 7.41 mm to (88.3, 109.2), turned to -90 degrees
- moved C18 7.06 mm to (87.6, 118.4), turned to -90 degrees
- moved R4 6.63 mm to (85.7, 109.2)
- moved C6 6.38 mm to (87.0, 97.2)
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Routing:
- net +5V: track 9.68 -> 45.9 mm, vias 0 -> 2
- net IN_C: track 0.00 -> 31.8 mm, vias 0 -> 1
- net IN_B: track 0.00 -> 30.0 mm, vias 0 -> 1
- net +12V: track 13.7 -> 43.1 mm, vias 6 -> 5
- net IN_A: track 0.00 -> 28.7 mm, vias 0 -> 1
- net GND: track 79.9 -> 52.5 mm, vias 42 -> 17
- net DC_Measure: track 12.1 -> 32.3 mm, vias 2 -> 1
- net B: track 1.24 -> 18.6 mm, vias 11 -> 2
- net Net-(U1-+): track 20.6 -> 5.68 mm, vias 2 -> 0
- net A: track 1.30 -> 16.1 mm, vias 11 -> 2
- net C: track 1.32 -> 15.4 mm, vias 11 -> 2
- net Shunt_1: track 12.0 -> 5.14 mm, vias 0 -> 1
- net Shunt_2: track 12.0 -> 5.78 mm, vias 99 -> 64
- net Net-(R2-Pad1): track 2.29 -> 6.58 mm, vias 0 -> 2
- net G4: track 5.02 -> 9.24 mm, vias 0 -> 1
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- added copper zone on In2.Cu, net +12V
- added copper zone on In1.Cu, net Enable
- removed copper zone on In1.Cu, net GND
- removed copper zone on In2.Cu, net GND
- removed copper zone on In3.Cu, net GND
- removed copper zone on In4.Cu, net GND
- removed copper zone on B.Cu, net Shunt_1
- removed copper zone on In1.Cu, net Shunt_1
- removed copper zone on In2.Cu, net Shunt_1
- removed copper zone on In3.Cu, net Shunt_1
- removed copper zone on In4.Cu, net Shunt_1
- removed copper zone on In2.Cu, net Shunt_2
- removed copper zone on In3.Cu, net Shunt_2
