File: Temperture.kicad_sch (KiCad schematic)
At the start: 6 parts

Commit message: Отчётная версия
Parts:
- renumbered C14 to C46, C30 to C47
Other:
- company: (none) -> Московский Политех
- moved on the sheet: C46, C47, C48, D2, D3, D4
