File: Силовая плата.kicad_sch (KiCad schematic)
At the start: 0 parts

Commit message: Отчётная версия
Other:
- added sheet Connection_List (Connection_List.kicad_sch)
- note added: "Схема электрическая"
- note added: "принципиальная"
- company: (none) -> Московский Политех
- title: (none) -> Узел силовой
Changed lines of the file:
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@@
 (kicad_sch (version 20230121) (generator eeschema)
   (paper "A4")
-  (sheet (at 77.47 19.05) (size 48.26 30.48) (fields_autoplaced)
+  (title_block
+    (title "Узел силовой")
+    (company "Московский Политех")
+    (comment 1 "МПСТ.76721.758764.01.Э3.М")
+    (comment 2 "Филатов")
+    (comment 3 "Нестеров")
+    (comment 4 "Келлер")
+    (comment 5 "Шевырев")
+    (comment 6 "Саяхов")
+  )
+  (text "Схема электрическая\n" (at 190.5 185.42 0)
+    (effects (font (size 2.5 2.5)) (justify left bottom))
+  )
+  (text "принципиальная\n" (at 194.31 187.96 0)
+    (effects (font (size 2.5 2.5)) (justify left bottom))
+  )
+  (sheet (at 81.28 35.56) (size 48.26 30.48) (fields_autoplaced)
     (stroke (width 0.1524) (type solid))
     (fill (color 0 0 0 0.0000))
-    (property "Sheetname" "Temperture" (at 77.47 18.3384 0)
-      (effects (font (size 1.27 1.27)) (justify left bottom))
+    (property "Sheetname" "Temperture" (at 81.28 34.2334 0)
+      (effects (font (size 2.5 2.5)) (justify left bottom))
     )
-    (property "Sheetfile" "Temperture.kicad_sch" (at 77.47 50.1146 0)
-      (effects (font (size 1.27 1.27)) (justify left top))
+    (property "Sheetfile" "Temperture.kicad_sch" (at 81.28 66.6246 0)
+      (effects (font (size 1.27 1.27)) (justify left top) hide)
     )
-    (property "Поле2" "" (at 77.47 19.05 0)
+    (property "Поле2" "" (at 81.28 35.56 0)
       (effects (font (size 1.27 1.27)) hide)
     )
     (instances
       (project "Силовая плата"
-        (path "/96c6fc92-8ec6-44f7-b0dc-9ad8f1acea09" (page "6"))
+        (path "/96c6fc92-8ec6-44f7-b0dc-9ad8f1acea09" (page "3"))
       )
     )
   )
-  (sheet (at 129.54 19.05) (size 48.26 30.48) (fields_autoplaced)
+  (sheet (at 133.35 35.56) (size 48.26 30.48) (fields_autoplaced)
     (stroke (width 0.1524) (type solid))
     (fill (color 0 0 0 0.0000))
-    (property "Sheetname" "Polarity_Protection" (at 129.54 18.3384 0)
-      (effects (font (size 1.27 1.27)) (justify left bottom))
+    (property "Sheetname" "Polarity_Protection" (at 133.35 34.2334 0)
+      (effects (font (size 2.5 2.5)) (justify left bottom))
     )
-    (property "Sheetfile" "Polarity_Protection.kicad_sch" (at 129.54 50.1146 0)
-      (effects (font (size 1.27 1.27)) (justify left top))
+    (property "Sheetfile" "Polarity_Protection.kicad_sch" (at 133.35 66.6246 0)
+      (effects (font (size 1.27 1.27)) (justify left top) hide)
     )
-    (property "Поле2" "" (at 129.54 19.05 0)
+    (property "Поле2" "" (at 133.35 35.56 0)
       (effects (font (size 1.27 1.27)) hide)
     )
-    (property "Поле3" "" (at 129.54 19.05 0)
+    (property "Поле3" "" (at 133.35 35.56 0)
       (effects (font (size 1.27 1.27)) hide)
     )
@@
     )
   )
-  (sheet (at 181.61 19.05) (size 48.26 30.48) (fields_autoplaced)
+  (sheet (at 185.42 35.56) (size 48.26 30.48) (fields_autoplaced)
     (stroke (width 0.1524) (type solid))
     (fill (color 0 0 0 0.0000))
-    (property "Sheetname" "Connector" (at 181.61 18.3384 0)
-      (effects (font (size 1.27 1.27)) (justify left bottom))
+    (property "Sheetname" "Connector" (at 185.42 34.2334 0)
+      (effects (font (size 2.5 2.5)) (justify left bottom))
     )
-    (property "Sheetfile" "Connector.kicad_sch" (at 181.61 50.1146 0)
-      (effects (font (size 1.27 1.27)) (justify left top))
+    (property "Sheetfile" "Connector.kicad_sch" (at 185.42 66.6246 0)
+      (effects (font (size 1.27 1.27)) (justify left top) hide)
     )
-    (property "Поле2" "" (at 181.61 19.05 0)
+    (property "Поле2" "" (at 185.42 35.56 0)
       (effects (font (size 1.27 1.27)) hide)
     )
@@
     )
   )
-  (sheet (at 25.4 19.05) (size 48.26 30.48) (fields_autoplaced)
+  (sheet (at 29.21 35.56) (size 48.26 30.48) (fields_autoplaced)
     (stroke (width 0.1524) (type solid))
     (fill (color 0 0 0 0.0000))
-    (property "Sheetname" "Power" (at 25.4 18.3384 0)
-      (effects (font (size 1.27 1.27)) (justify left bottom))
+    (property "Sheetname" "Power" (at 29.21 34.2334 0)
+      (effects (font (size 2.5 2.5)) (justify left bottom))
     )
-    (property "Sheetfile" "Power.kicad_sch" (at 25.4 50.1146 0)
-      (effects (font (size 1.27 1.27)) (justify left top))
+    (property "Sheetfile" "Power.kicad_sch" (at 29.21 66.6246 0)
+      (effects (font (size 1.27 1.27)) (justify left top) hide)
     )
     (instances
@@
       )
     )
+  )
+  (sheet (at 237.49 35.56) (size 48.26 30.48) (fields_autoplaced)
+    (stroke (width 0.1524) (type solid))
+    (fill (color 0 0 0 0.0000))
+    (property "Sheetname" "Connection_List" (at 237.49 34.2334 0)
+      (effects (font (size 2.5 2.5)) (justify left bottom))
+    )
+    (property "Sheetfile" "Connection_List.kicad_sch" (at 237.49 66.6246 0)
+      (effects (font (size 1.27 1.27)) (justify left top) hide)
+    )
+    (property "Поле2" "" (at 237.49 35.56 0)
+      (effects (font (size 1.27 1.27)) hide)
+    )
+    (instances
+      (project "Силовая плата"
+        (path "/96c6fc92-8ec6-44f7-b0dc-9ad8f1acea09" (page "6"))
+      )
+    )
