File: Connection_List.kicad_sch (KiCad schematic)
At the start: 0 parts

Commit message: Изменения: добавил папку с отчетностью
Other:
- note added: "A1"
- note added: "A3"
- note added: "Узел силовой"
- note added: "Узел соединительный"
